File: flashlight-bottom.sch (EAGLE design)
At the start: 1 part, among them SW1 DIL3-TOGGLE-SWITCHDIL3

Commit message: rev 2.0 of the bottom board, plus minor tweaks to the top board
Parts:
- removed SW1: DIL3-TOGGLE-SWITCHDIL3, chrisy-components:DIL3-TOGGLE-SWITCHDIL3
Changed lines of the file:
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@@
 <?xml version="1.0" encoding="utf-8"?>
 <!DOCTYPE eagle SYSTEM "eagle.dtd">
-<eagle version="7.1.0">
+<eagle version="7.2.0">
 <drawing>
 <settings>
@@
 <setting verticaltext="up"/>
 </settings>
-<grid distance="0.1" unitdist="inch" unit="inch" style="lines" multiple="1" display="yes" altdistance="0.01" altunitdist="inch" altunit="inch"/>
+<grid distance="0.1" unitdist="inch" unit="inch" style="lines" multiple="1" display="no" altdistance="0.01" altunitdist="inch" altunit="inch"/>
 <layers>
 <layer number="1" name="Top" color="4" fill="1" visible="no" active="no"/>
@@
 </classes>
 <parts>
-<part name="SW1" library="chrisy-components" deviceset="DIL3-TOGGLE-SWITCH" device="DIL3"/>
 </parts>
 <sheets>
@@
 </plain>
 <instances>
-<instance part="SW1" gate="G$1" x="30.48" y="30.48"/>
 </instances>
 <busses>
